Commit message: Commit_first_try_on_real_robot

File: src/abb_irb140_support/urdf/irb140.urdf (robot description, URDF)
Before this commit: robot abb_irb140, 12 links, 11 joints
Links:
- removed link obj_position_link
Joints:
- removed joint plane_link-obj_position_link

File: src/abb_irb140_support/urdf/irb140_macro.xacro (robot description, xacro)
@@ -243,5 +243,5 @@
     <child link="obj_position_link"/>
   </joint> -->
-  <link name="${prefix}obj_position_link">
+  <!-- <link name="${prefix}obj_position_link">
     <visual>
       <origin rpy="0 0 0" xyz="0 0 0.1"/>
@@ -261,8 +261,8 @@
   </link>
   <joint name="${prefix}base_link-obj_position_link" type="fixed">
-    <origin rpy="0 0 0" xyz="0.4 0 0"/>
+    <origin rpy="0 0 0" xyz="0.5 0 0"/>
     <parent link="${prefix}base_link"/>
     <child link="${prefix}obj_position_link"/>
-  </joint>
+  </joint> -->
 </xacro:macro>
 </robot>
