Commit message: Camera-offset

File: src/abb_irb140_support/urdf/camera.xacro (robot description, xacro)
@@ -2,5 +2,5 @@
 <robot xmlns:xacro="http://www.ros.org/wiki/xacro" >
     <joint name="camera_joint" type="fixed">
-        <parent link="tool0"/>
+        <parent link="tool1"/>
         <child link="camera_link"/>
         <origin xyz="0 0 0" rpy="0 0 0"/>
@@ -9,9 +9,10 @@
         <visual>
             <geometry>
-                <box size="0.010 0.03 0.03"/>
+                <box size="0.0 0.0 0.0"/>
+                <!-- <box size="0.010 0.03 0.03"/> -->
             </geometry>
-            <material name="blue">
+            <!-- <material name="blue">
                 <color rgba="0 0 1 1"/>
-            </material>
+            </material> -->
         </visual>
     </link>
@@ -23,5 +24,5 @@
     <link name="camera_link_optical"></link>
     <gazebo reference="camera_link">
-        <material>Gazebo/Red</material>
+        <material>Gazebo/Green</material>
         <sensor name="camera" type="camera">
             <pose> 0 0 0 0 0 0 </pose>

File: src/abb_irb140_support/urdf/irb140.urdf (robot description, URDF)
Before this commit: robot abb_irb140, 11 links, 10 joints
Links:
- added link tool1
- link tool0: geometry collision mesh filename=package://abb_irb140_support/meshes/irb140/visual/tool0.stl scale=0.01 0.01 0.01; visual mesh filename=package://abb_irb140_support/meshes/irb140/visual/tool0.stl scale=0.01 0.01 0.01
Joints:
- added joint tool0-tool1: type fixed, parent tool0, child tool1, origin xyz=0 0 0 rpy=3.14159 1.5708 0
- joint base_link-wall_link: origin xyz=-0.6 0 0 rpy=0 0 0 -> xyz=-0.57 0 0 rpy=0 0 0
- joint joint_6-tool0: origin xyz=0 0 0 rpy=0 0 0 -> xyz=0.101 0.022 -0.023 rpy=0 0 0

File: src/abb_irb140_support/urdf/irb140.xacro (robot description, xacro)
@@ -1,4 +1,8 @@
 <?xml version="1.0" ?>
 <robot name="abb_irb140" xmlns:xacro="http://ros.org/wiki/xacro">
+	<!-- <xacro:arg name="param_height" default="0.265" />
+	<xacro:arg name="param_width" default="0.23" />
+	<xacro:arg name="param_length" default="0.07" />
+	<xacro:arg name="param_center" default="0.5" /> -->
 	<xacro:include filename="$(find abb_irb140_support)/urdf/irb140_macro.xacro"/>
 	<xacro:abb_irb140 prefix=""/>

File: src/abb_irb140_support/urdf/irb140_macro.xacro (robot description, xacro)
@@ -2,4 +2,8 @@
 <robot xmlns:xacro="http://ros.org/wiki/xacro">
 <xacro:include filename="camera.xacro" />
+<!-- <xacro:property name="param_height" value="0.265" />
+<xacro:property name="param_width" value="0.23" />
+<xacro:property name="param_length" value="0.07" />
+<xacro:property name="param_center" value="0.5" /> -->
 <!-- <xacro:macro name="abb_irb140" params="prefix param_value"> -->
 <!-- <xacro:include filename="$(find abb_irb140_support)/config/parameters.yaml" /> -->
@@ -157,5 +161,49 @@
     </collision>
   </link>
-  <link name="${prefix}tool0"/>
+  <!-- <link name="${prefix}tool0">
+    <visual>
+      <origin rpy="0 0 0" xyz="-0.515 0.001 -0.181"/>
+      <geometry>
+        <mesh filename="package://abb_irb140_support/meshes/irb140/visual/tool0.stl" scale="0.001 0.001 0.001"/>
+      </geometry>
+      <material name="green">
+        <color rgba="0 1 0 1"/>
+      </material>
+    </visual>
+    <collision>
+      <origin rpy="0 0 0" xyz="-0.515 0.001 -0.181"/>
+      <geometry>
+        <mesh filename="package://abb_irb140_support/meshes/irb140/collision/tool0.stl" scale="0.001 0.001 0.001"/>
+      </geometry>
+      <material name="green">
+        <color rgba="0 1 0 1"/>
+      </material>
+    </collision>
+  </link> -->
+  <link name="${prefix}tool0">
+    <visual>
+    <origin rpy="0 0 0" xyz="-0.5945 -0.022 -0.6879"/>
+      <!-- <origin rpy="0 0 0" xyz="-0.5845 -0.0234 -0.765"/> fail -->
+      <!-- <origin rpy="0 0 0" xyz="-0.12145 -0.0234 -0.765"/> -->
+      <!-- <origin rpy="0 -1.5708 0" xyz="-0.5145 0 -0.711"/> -->
+      <geometry>
+        <mesh filename="package://abb_irb140_support/meshes/irb140/visual/tool0.stl" scale="0.01 0.01 0.01"/>
+      </geometry>
+      <material name="green">
+        <color rgba="0 1 0 1"/>
+      </material>
+    </visual>
+    <collision>
+      <origin rpy="0 0 0" xyz="-0.5945 -0.022 -0.6879"/>
+      <!-- <origin rpy="0 0 0" xyz="-0.5145 0 -0.711"/> -->
+      <geometry>
+        <mesh filename="package://abb_irb140_support/meshes/irb140/visual/tool0.stl" scale="0.01 0.01 0.01"/>
+      </geometry>
+      <material name="green">
+        <color rgba="0 1 0 1"/>
+      </material>
+    </collision>
+  </link>
+  <link name="${prefix}tool1"/>
     <!-- end of link list -->
     <!-- joint list -->
@@ -211,5 +259,10 @@
     <parent link="${prefix}link_6"/>
     <child link="${prefix}tool0"/>
-    <origin rpy="0 0 0" xyz="0 0 0"/>
+    <origin rpy="0 0 0" xyz="0.08 0.022 -0.023"/>
+  </joint>
+  <joint name="${prefix}tool-tool1" type="fixed">
+    <parent link="tool0"/>
+    <child link="tool1"/>
+    <origin rpy="3.14159 1.5708 0" xyz="0 0 0"/>
   </joint>
     <!-- end of joint list -->
@@ -223,24 +276,68 @@
   <!-- <link name="obj_position_link">
     <visual>
-      <origin rpy="0 0 0" xyz="0 0 $(param_value)"/>
-      <geometry>
-        <box size="$(param_length) $(param_width) $(param_height)"/>
-      </geometry>
-      <material name="green">
-        <color rgba="0 1 0 1"/>
-      </material>
-    </visual>
-    <collision>
-      <origin rpy="0 0 0" xyz="0 0 $(param_value)"/>
-      <geometry>
-        <box size="$(param_length) $(param_width) $(param_height)"/>
-      </geometry>
-    </collision>
-  </link>
-  <joint name="base_link-obj_position_link" type="fixed">
-    <origin rpy="0 0 0" xyz="$(param_center) 0 0"/>
+      <origin rpy="0 0 0" xyz="0 0 ${param_height/2}"/>
+      <geometry>
+        <box size="${param_length} ${param_width} ${param_height}"/>
+      </geometry>
+      <material name="green">
+        <color rgba="0 1 0 1"/>
+      </material>
+    </visual>
+    <collision>
+      <origin rpy="0 0 0" xyz="0 0 ${param_height/2}"/>
+      <geometry>
+        <box size="${param_length} ${param_width} ${param_height}"/>
+      </geometry>
+    </collision>
+  </link> -->
+  <!-- <joint name="base_link-obj_position_link" type="fixed">
+    <origin rpy="0 0 0" xyz="${param_center} 0 0"/>
     <parent link="base_link"/>
     <child link="obj_position_link"/>
   </joint> -->
+  <link name="obj_position_link">
+    <visual>
+        <origin rpy="0 0 0" xyz="0 0 $(arg param_value)"/>
+        <geometry>
+            <box size="$(arg param_length) $(arg param_width) $(arg param_height)"/>
+        </geometry>
+        <material name="green">
+            <color rgba="0 1 0 1"/>
+        </material>
+    </visual>
+    <collision>
+        <origin rpy="0 0 0" xyz="0 0 $(arg param_value)"/>
+        <geometry>
+            <box size="$(arg param_length) $(arg param_width) $(arg param_height)"/>
+        </geometry>
+    </collision>
+</link>
+<joint name="base_link-obj_position_link" type="fixed">
+    <origin rpy="0 0 0" xyz="$(arg param_center) 0 0"/>
+    <parent link="base_link"/>
+    <child link="obj_position_link"/>
+</joint>
+  <!-- <link name="${prefix}holder_link">
+    <visual>
+      <origin rpy="0 0 0" xyz="0 0 0.15"/>
+      <geometry>
+        <box size="0.05 0.05 0.3"/>
+      </geometry>
+      <material name="green">
+        <color rgba="0 1 0 1"/>
+      </material>
+    </visual>
+    <collision>
+      <origin rpy="0 0 0" xyz="0 0 0.15"/>
+      <geometry>
+        <box size="0.05 0.05 0.3"/>
+      </geometry>
+    </collision>
+  </link>
+  <joint name="${prefix}base_link-holder_link" type="fixed">
+    <origin rpy="0 0 0" xyz="0.3 0 0"/>
+    <parent link="${prefix}base_link"/>
+    <child link="${prefix}holder_link"/>
+  </joint> -->
   <!-- <link name="${prefix}obj_position_link">
     <visual>
@@ -259,7 +356,7 @@
       </geometry>
     </collision>
-  </link>
-  <joint name="${prefix}base_link-obj_position_link" type="fixed">
-    <origin rpy="0 0 0" xyz="0.5 0 0"/>
+  </link> -->
+  <!-- <joint name="${prefix}base_link-obj_position_link" type="fixed">
+    <origin rpy="0 0 0" xyz="${param_center} 0 0"/>
     <parent link="${prefix}base_link"/>
     <child link="${prefix}obj_position_link"/>
